File: ASM2022.sch (EAGLE design)
At the start: 42 parts, among them J1 SM02B-SRSS-TB(LF)(SN), J2 47346-0001, J3 EVP-ANDA1A, J4 EVP-ANDA1A, J5 EVP-ANDA1A, J6 DF12-32-DP, J7 EVP-ANDA1A, Q1 DMP2035U, SW1 PCM12SMTR, U1 XC6210B33, U2 MCP73831, U3 UG-9664HDDAG01, U4 FAN5340, U5 ATSAMD21G18A, Y1 32.7680

Commit message: Update to Rev 4 PCB
Parts:
- added R10: 1.00M, tinycircuits:AS-ITM-00005
- added R11: 1.2M, tinycircuits:AS-ITM-00280
- C1: value 4.7uF -> 10uF; device tinycircuits:AS-ITM-00088 -> tinycircuits:AS-ITM-00002; PARTNO AS-ITM-00088 -> AS-ITM-00002; VALUE 4.7uF -> 10uF
- C10: VALUE 10uF -> (none)
- C11: value .1uF -> 10uF; device tinycircuits:AS-ITM-00008 -> tinycircuits:AS-ITM-00002; PARTNO AS-ITM-00008 -> AS-ITM-00002
- C12: value .1uF -> 10uF; device tinycircuits:AS-ITM-00008 -> tinycircuits:AS-ITM-00045; PARTNO AS-ITM-00008 -> AS-ITM-00045; VALUE 0.1uF -> 10uF
- C13: value .1uF -> 10uF; device tinycircuits:AS-ITM-00008 -> tinycircuits:AS-ITM-00002; PARTNO AS-ITM-00008 -> AS-ITM-00002; VALUE 0.1uF -> 10uF
- C14: value .1uF -> 4.7uF; device tinycircuits:AS-ITM-00008 -> tinycircuits:AS-ITM-00232; PARTNO AS-ITM-00008 -> AS-ITM-00232; VALUE 0.1uF -> F931D475MAA
- C2: value 10uF -> 22pF; device tinycircuits:AS-ITM-00045 -> tinycircuits:AS-ITM-00211; PARTNO AS-ITM-00045 -> AS-ITM-00211; VALUE (none) -> 22pF
- C3: value 10uF -> 22pF; device tinycircuits:AS-ITM-00002 -> tinycircuits:AS-ITM-00211; PARTNO AS-ITM-00002 -> AS-ITM-00211; VALUE 10uF -> 22pF
- C4: value 10uF -> .1uF; device tinycircuits:AS-ITM-00002 -> tinycircuits:AS-ITM-00008; PARTNO AS-ITM-00002 -> AS-ITM-00008
- C5, C7: value 22pF -> .1uF; device tinycircuits:AS-ITM-00211 -> tinycircuits:AS-ITM-00008; PARTNO AS-ITM-00211 -> AS-ITM-00008; VALUE 22pF -> 0.1uF
- C6: device tinycircuits:AS-ITM-00232 -> tinycircuits:AS-ITM-00088; PARTNO AS-ITM-00232 -> AS-ITM-00088; VALUE F931D475MAA -> 4.7uF
- C8: value 4.7uF -> .1uF; device tinycircuits:AS-ITM-00242 -> tinycircuits:AS-ITM-00008; PARTNO (none) -> AS-ITM-00008; VALUE (none) -> 0.1uF
- D1: value MBR120 -> AMBER; device tinycircuits:AS-ITM-00111 -> tinycircuits:AS-ITM-00026; PARTNO (none) -> AS-ITM-00026; VALUE (none) -> AMBER
- D2: value AMBER -> CD0603; device tinycircuits:AS-ITM-00026 -> tinycircuits:AS-ITM-00009; PARTNO AS-ITM-00026 -> AS-ITM-00009; VALUE AMBER -> (none)
- D3: value CD0603 -> MBR120; device tinycircuits:AS-ITM-00009 -> tinycircuits:AS-ITM-00111; PARTNO AS-ITM-00009 -> (none)
- J1: value SM02B-SRSS-TB(LF)(SN) -> 47346-0001; device tinycircuits:AS-ITM-00231 -> tinycircuits:AS-ITM-00021
- J2: value 47346-0001 -> DF12-32-DP; device tinycircuits:AS-ITM-00021 -> tinycircuits:AS-ITM-00015; PARTNO (none) -> AS-ITM-00015; VALUE (none) -> DF12-32-DP
- J3: value EVP-ANDA1A -> SM02B-SRSS; device tinycircuits:AS-ITM-00236 -> tinycircuits:AS-ITM-00231; PARTNO AS-ITM-00236 -> (none); VALUE PTS840 GKP -> (none)
- J4, J5, J7: value EVP-ANDA1A -> PTS840GKP
- J6: value DF12-32-DP -> PTS840GKP; device tinycircuits:AS-ITM-00015 -> tinycircuits:AS-ITM-00236; PARTNO AS-ITM-00015 -> AS-ITM-00236; VALUE DF12-32-DP -> PTS840 GKP
- L1: PARTNO AS-ITM-00281 -> (none); VALUE 22uH -> (none)
- R1: value 5K -> 10K; device tinycircuits:AS-ITM-00289 -> tinycircuits:AS-ITM-00032; PARTNO (none) -> AS-ITM-00032
- R3: value 100k -> 10K; device tinycircuits:AS-ITM-00004 -> tinycircuits:AS-ITM-00032; PARTNO AS-ITM-00004 -> AS-ITM-00032; VALUE (none) -> 10.0K
- R4: value 1.2M -> 5K; device tinycircuits:AS-ITM-00280 -> tinycircuits:AS-ITM-00289; PARTNO AS-ITM-00280 -> (none); VALUE 1.2M -> (none)
- R5: value 115k -> 100k; device tinycircuits:AS-ITM-00179 -> tinycircuits:AS-ITM-00004; PARTNO (none) -> AS-ITM-00004; VALUE 115K -> (none)
- R6: value 4.7k -> 10K; device tinycircuits:AS-ITM-00167 -> tinycircuits:AS-ITM-00032; PARTNO AS-ITM-00167 -> AS-ITM-00032; VALUE 4.7K -> (none)
- R7, R9: value 10K -> 1.00M; device tinycircuits:AS-ITM-00032 -> tinycircuits:AS-ITM-00005; PARTNO AS-ITM-00032 -> AS-ITM-00005; VALUE (none) -> 1.00M
- R8: value 10K -> 16K; device tinycircuits:AS-ITM-00032 -> tinycircuits:AS-ITM-00314; PARTNO AS-ITM-00032 -> AS-ITM-00314; VALUE 10.0K -> 16K
- U1: value XC6210B33 -> MCP73831; device tinycircuits:AS-ITM-00046 -> tinycircuits:AS-ITM-00136
- U2: value MCP73831 -> ATSAMD21G18A; device tinycircuits:AS-ITM-00136 -> tinycircuits:AS-ITM-00273; PARTNO (none) -> AS-ITM-00273
- U3: value UG-9664HDDAG01 -> XC6210B33; device tinycircuits:AS-ITM-00158 -> tinycircuits:AS-ITM-00046
- U4: value FAN5340 -> AP3036B; device tinycircuits:AS-ITM-00277 -> tinycircuits:AS-ITM-00377; PARTNO (none) -> AS-ITM-00377; VALUE (none) -> AP3036B
- U5: value ATSAMD21G18A -> UG-9664HDDAG01; device tinycircuits:AS-ITM-00273 -> tinycircuits:AS-ITM-00158; PARTNO AS-ITM-00273 -> (none)
Connections:
- removed net AD4/SDA: J6.3, R8.1, U5.PA22
- removed net AD5/SCL: J6.1, R7.1, U5.PA23
- removed net N$13: R5.1, U4.VLED
- new net SCL: J2.1, R1.1, U2.PA23
- new net SDA: J2.3, R3.1, U2.PA22
- net +12V: now also C12.1, R7.2, U5.VCC; no longer C10.1, U3.VCC
- net +3V3: now also J2.6; no longer J6.6
- net +5V: now also C1.1, D3.A, J1.1, J2.8, R5.2, U1.VDD; no longer C3.1, D2.A, J2.1, J6.8, R3.2, U2.VDD
- net AD0: now also J2.11, U2.PA02; no longer J6.11, U5.PA02
- net AD1: now also J2.9, U2.PB08; no longer J6.9, U5.PB08
- net AD2: now also J2.7, U2.PB09; no longer J6.7, U5.PB09
- net AD3: now also J2.5, U2.PA04; no longer J6.5, U5.PA04
- net AD4: now also R10.2, R9.1, U2.PA05; no longer U5.PA05
- net AD5: now also J4.1, U2.PB02; no longer J3.1, U5.PB02
- net AREF: now also J2.13, U2.PA03; no longer J6.13, U5.PA03
- net ATN/IO38: now also U2.PA13, U5.CS#; no longer U3.CS#, U5.PA13
- net DBG_RXD: now also U2.PB23; no longer U5.PB23
- net DBG_TXD: now also J6.1, U2.PB22; no longer J5.1, U5.PB22
- net GND: now also J1.5, J1.P1, J1.P2, J1.P3, J1.P4, J1.P5, J1.P6, J2.12, J2.14, J6.2, R10.1, R11.1, R4.2, R5.1, R8.1, U2.GND1, U2.GND2, U2.GND3, U2.GNDANA, U5.BS1, U5.BS2, U5.D3, U5.D4, U5.D5, U5.D6, U5.D7, U5.E, U5.R/W#, U5.VSS; no longer J1.2, J2.5, J2.P1, J2.P2, J2.P3, J2.P4, J2.P5, J2.P6, J6.12, J6.14, R1.2, R3.1, R4.1, R6.1, U2.VSS, U3.BS1, U3.BS2, U3.D3, U3.D4, U3.D5, U3.D6, U3.D7, U3.E, U3.R/W#, U4.PGND, U5.GND1, U5.GND2, U5.GND3, U5.GNDANA
- net IO0: now also J2.24, U2.PA11; no longer J6.24, U5.PA11
- net IO1: now also J2.26, U2.PA10; no longer J6.26, U5.PA10
- net IO2: now also J2.28, U2.PA14; no longer J6.28, U5.PA14
- net IO3: now also J2.30, U2.PA09; no longer J6.30, U5.PA09
- net IO4: now also J2.32, U2.PA08; no longer J6.32, U5.PA08
- net IO5: now also J2.31, U2.PA15; no longer J6.31, U5.PA15
- net IO6: now also J2.29, U2.PA20; no longer J6.29, U5.PA20
- net IO7: now also J2.27, U2.PA21; no longer J6.27, U5.PA21
- net IO8: now also J2.25, U2.PA06; no longer J6.25, U5.PA06
- net IO9: now also J2.23, U2.PA07; no longer J6.23, U5.PA07
- net MISO: now also J2.17, U2.PA19; no longer J6.17, U5.PA19
- net MISO_ALT: now also U2.PA12, U5.D/C#; no longer U3.D/C#, U5.PA12
- net MOSI: now also J2.19, U2.PA16; no longer J6.19, U5.PA16
- net MOSI_ALT: now also U2.PB10, U5.D1; no longer U3.D1, U5.PB10
- net N$1: now also C2.1, U2.PA00; no longer C5.1, U5.PA00
- net N$11: now also R11.2, U5.IREF; no longer R4.2, U3.IREF
- net N$12: now also C14.1, U5.VCOMH; no longer C6.1, U3.VCOMH
- net N$15: now also U5.D2; no longer U3.D2
- net N$2: now also D3.C; no longer D1.C
- net N$3: now also C3.1, U2.PA01; no longer C7.1, U5.PA01
- net N$5: now also D1.C; no longer D2.C
- net N$6: now also R4.1, U1.PROG; no longer R1.1, U2.PROG
- net N$7: now also U1.STAT; no longer U2.STAT
- net N$8: now also U2.VDDCORE; no longer U5.VDDCORE
- net RESET: now also D2.A, J2.22, R6.1, U2.RESETN; no longer D3.A, J6.22, R9.1, U5.RESETN
- net RSV2: now also J2.16; no longer J6.16
- net RX_LED/IO25/AIN11: now also J5.1, U2.PB03; no longer J4.1, U5.PB03
- net SCK: now also J2.15, U2.PA17; no longer J6.15, U5.PA17
- net SCK_ALT: now also U2.PB11, U5.D0; no longer U3.D0, U5.PB11
- net SS: now also J2.21, U2.PA18; no longer J6.21, U5.PA18
- net SWCLK: now also J2.20, U2.PA30; no longer J6.20, U5.PA30
- net SWDIO: now also J2.18, U2.PA31; no longer J6.18, U5.PA31
- net TX_LED/IO26: now also U2.PA27, U5.RES#; no longer U3.RES#, U5.PA27
- net USB_HOST_EN/IO27: now also U2.PA28, U4.CTRL; no longer U4.SHDN, U5.PA28
- net USB_N: now also J1.2, U2.PA24; no longer J2.2, U5.PA24
- net USB_P: now also J1.3, U2.PA25; no longer J2.3, U5.PA25
- net VBATT: now also C6.1, J2.4, J3.1, R9.2, U1.VBAT; no longer C1.1, J1.1, J6.4, U2.VBAT
- net VCC: now also C5.1, C7.1, C8.1, D2.C, J2.2, R1.2, R3.2, R6.2, U2.VDDANA, U2.VDDIN, U2.VDDIO1, U2.VDDIO2, U3.VOUT, U5.VDD, U5.VDDIO; no longer C12.1, C13.1, C14.1, D3.C, J6.2, R7.2, R8.2, R9.2, U1.VOUT, U3.VDD, U3.VDDIO, U5.VDDANA, U5.VDDIN, U5.VDDIO1, U5.VDDIO2
- net VCC_IN: now also C10.1, C13.1, U3.CE, U3.VIN; no longer C2.1, C8.1, U1.CE, U1.VIN
- net VIN: now also J2.10; no longer J6.10
- net V_FB: now also R7.1, R8.2; no longer R5.2, R6.2
Other:
- note added: "4"
- note removed: "3"
- moved on the sheet: C1, C10, C11, C12, C13, C14, C2, C3, C4, C5, C6, C7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
